File: 5v levelshifter board/5v levelshifter board.kicad_pcb (KiCad board)
At the start: 2 copper layers, 63.5 x 78.7 mm, 45 parts, among them IC1 MAX3002EUP+T, IC2 MAX3002EUP+T, IC3 MAX3002EUP+T, IC4 MAX3002EUP+T, IC5 MAX3002EUP+T, IC6 MAX3002EUP+T, IC7 MAX3002EUP+T, IC8 MAX3002EUP+T, J1 5v coupling, J10 48-55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

Commit message: revised board design and added gerber files
Parts:
- added G***: LOGO, Evan's parts:pcbway logo, B.Cu at (151.8, 143.5)
- moved G*** 12.3 mm to (141.6, 132.1)
Routing:
- net 5v_32: track 23.7 -> 20.3 mm
- net 5v_33: track 22.0 -> 18.7 mm
- net 5v_34: track 20.1 -> 17.9 mm
- net 5v_35: track 18.2 -> 17.1 mm
- net 5v_40: track 11.8 -> 12.6 mm
Other:
- board text added: "3.3v"
- board text added: "5v"
- board text added: "RST"
- board text added: "TCK"
- board text added: "TDI"
- board text added: "TDO"
- board text added: "TMS"
- board text added: "Vjtag"
